Commit message: added lidar

File: models/robot/sentry_robot_v2.urdf.xacro (robot description, xacro)
@@ -56,4 +56,7 @@
 	    </collision>
 	  </link>
+	<gazebo reference="sentry_base_link">
+   		<material> Gazebo/Blue</material>
+    </gazebo>
   	</xacro:macro>
 	<xacro:macro name="mecanum_wheel" params="prefix parent *origin reflect">
